File: AudioInterface.sch (KiCad schematic (older format))
At the start: 4 parts, among them J3 REM/DATA, U3 HS-100B

Commit message: Add BOM and clarify some footprints
Parts:
- C11: footprint Capacitor_SMD:CP_Elec_4x3 -> Capacitor_SMD:C_1210_3225Metric; Manufacturer_Name (none) -> AVX; Manufacturer_Part_Number (none) -> TPST107M004R0500; Price (none) -> 0.93; Vendor (none) -> Mouser; Vendor Part Number (none) -> 581-TPST107M004R0500
- C12: footprint Capacitor_SMD:CP_Elec_4x3 -> Capacitor_SMD:C_1210_3225Metric; Manufacturer_Name (none) -> Walsin; Manufacturer_Part_Number (none) -> 1210F106Z100CT; Price (none) -> 0.29; Vendor (none) -> Mouser; Vendor Part Number (none) -> 791-1210F106Z100CT
- J3: Description (none) -> TX-500 REM/DATA Interconnect; Manufacturer_Name (none) -> JST; Manufacturer_Part_Number (none) -> B3B-PH-SM4-TB; Price (none) -> 0.35; Vendor (none) -> Mouser; Vendor Part Number (none) -> 485-4389
- U3: Description LQFP-48 Video-Audio Interface ICs RoHS -> USB Audio Interface; Manufacturer_Name cmedia -> Cmedia; Price (none) -> 0.78; Vendor (none) -> Symmetry; Vendor Part Number (none) -> HS-100B
Changed lines of the file:
@@
 F 1 "HS-100B" H 4500 3700 50  0000 L CNN
 F 2 "Package_QFP:LQFP-48_7x7mm_P0.5mm" H 6350 3950 50  0001 L CNN
-F 3 "https://datasheet.lcsc.com/szlcsc/1906061502_Cmedia-HS-100B_C371351.pdf" H 6350 3850 50  0001 L CNN
-F 4 "LQFP-48 Video-Audio Interface ICs RoHS" H 6350 3750 50  0001 L CNN "Description"
+F 3 "1.6" H 6350 3850 50  0001 L CNN
+F 4 "USB Audio Interface" H 6350 3750 50  0001 L CNN "Description"
 F 5 "1.6" H 6350 3650 50  0001 L CNN "Height"
-F 6 "cmedia" H 6350 3550 50  0001 L CNN "Manufacturer_Name"
+F 6 "Cmedia" H 6350 3550 50  0001 L CNN "Manufacturer_Name"
 F 7 "HS-100B" H 6350 3450 50  0001 L CNN "Manufacturer_Part_Number"
-F 8 "" H 6350 3350 50  0001 L CNN "Mouser Part Number"
-F 9 "" H 6350 3250 50  0001 L CNN "Mouser Price/Stock"
-F 10 "" H 6350 3150 50  0001 L CNN "Arrow Part Number"
-F 11 "" H 6350 3050 50  0001 L CNN "Arrow Price/Stock"
+F 8 "0.78" H 4600 3900 50  0001 C CNN "Price"
+F 9 "HS-100B" H 4600 3900 50  0001 C CNN "Vendor Part Number"
+F 10 "Symmetry" H 4600 3900 50  0001 C CNN "Vendor"
 	1    4800 3350
 	1    0    0    -1
@@
 F 1 "REM/DATA" H 8172 3433 50  0000 R CNN
 F 2 "Connector_JST:JST_PH_B3B-PH-SM4-TB_1x03-1MP_P2.00mm_Vertical" H 8200 3500 50  0001 C CNN
-F 3 "~" H 8200 3500 50  0001 C CNN
+F 3 "https://www.mouser.com/datasheet/2/737/4389_C13924-001_CCP-W20-03-BK-SMT-R-A-1708610.pdf" H 8200 3500 50  0001 C CNN
+F 4 "TX-500 REM/DATA Interconnect" H 8172 3624 50  0001 C CNN "Description"
+F 5 "JST" H 8172 3624 50  0001 C CNN "Manufacturer_Name"
+F 6 "B3B-PH-SM4-TB" H 8172 3624 50  0001 C CNN "Manufacturer_Part_Number"
+F 7 "0.35" H 8172 3624 50  0001 C CNN "Price"
+F 8 "485-4389" H 8172 3624 50  0001 C CNN "Vendor Part Number"
+F 9 "Mouser" H 8172 3624 50  0001 C CNN "Vendor"
 	1    8200 3500
 	-1   0    0    -1
@@
 	1    0    0    -1
 $EndComp
-Wire Wire Line
-	6500 3350 6650 3350
-Wire Wire Line
-	6650 3350 6650 3650
-Wire Wire Line
-	6500 3650 6650 3650
-Connection ~ 6650 3650
-Wire Wire Line
-	6650 3650 6650 4450
-Wire Wire Line
-	6500 4450 6650 4450
-Connection ~ 6650 4450
-Wire Wire Line
-	6650 4450 6650 4650
 $Comp
 L power:GNDREF #PWR0111
@@
 	1    0    0    -1
 $EndComp
-Wire Wire Line
-	4800 4450 4600 4450
-Wire Wire Line
-	6500 4150 7450 4150
-Wire Wire Line
-	7450 4150 7450 3500
-Wire Wire Line
-	7450 3500 8000 3500
-Wire Wire Line
-	6500 3950 7250 3950
-Wire Wire Line
-	7250 3950 7250 3750
-Wire Wire Line
-	6500 3750 7250 3750
-Connection ~ 7250 3750
 $Comp
 L power:VBUS #PWR0112
@@
 	1    0    0    -1
 $EndComp
-Wire Wire Line
-	6500 3450 6900 3450
-Wire Wire Line
-	6500 3550 6900 3550
-Wire Wire Line
-	6900 3550 6900 3450
-Wire Wire Line
-	6500 4050 6900 4050
-Wire Wire Line
-	6900 4050 6900 3550
-Connection ~ 6900 3550
-Wire Wire Line
-	5800 5250 5800 5400
-Wire Wire Line
-	5800 5400 4600 5400
-Wire Wire Line
-	4600 4450 4600 5400
-Wire Wire Line
-	4600 5400 4600 5500
-Connection ~ 4600 5400
-Wire Wire Line
-	4800 4250 4600 4250
-Wire Wire Line
-	4600 4250 4600 4450
-Connection ~ 4600 4450
-Wire Wire Line
-	4800 4050 4400 4050
-Wire Wire Line
-	4400 4050 4400 3850
-Wire Wire Line
-	4400 3850 4800 3850
-Wire Wire Line
-	5900 2550 5900 2350
-Wire Wire Line
-	5900 2350 6650 2350
-Wire Wire Line
-	6650 2350 6650 3350
-Connection ~ 6650 3350
-Text Notes 5400 1700 0    50   ~ 0
-See HS-100B datasheet
-Text Notes 8100 3150 0    50   ~ 0
-See TX-500 adapters\nAudio data cable
 $Comp
 L Device:CP C12
@@
 F 0 "C12" V 7395 3300 50  0000 C CNN
 F 1 "10μF" V 7486 3300 50  0000 C CNN
-F 2 "Capacitor_SMD:CP_Elec_4x3" H 7688 3150 50  0001 C CNN
-F 3 "~" H 7650 3300 50  0001 C CNN
+F 2 "Capacitor_SMD:C_1210_3225Metric" H 7688 3150 50  0001 C CNN
+F 3 "https://www.mouser.com/datasheet/2/210/WTC_MLCC_General_Purpose-1534899.pdf" H 7650 3300 50  0001 C CNN
+F 4 "Walsin" H 7395 3400 50  0001 C CNN "Manufacturer_Name"
+F 5 "1210F106Z100CT" H 7395 3400 50  0001 C CNN "Manufacturer_Part_Number"
+F 6 "0.29" H 7395 3400 50  0001 C CNN "Price"
+F 7 "791-1210F106Z100CT" H 7395 3400 50  0001 C CNN "Vendor Part Number"
+F 8 "Mouser" H 7395 3400 50  0001 C CNN "Vendor"
 	1    7650 3300
 	0    1    1    0
 $EndComp
-Wire Wire Line
-	7250 3300 7500 3300
-Wire Wire Line
-	7250 3300 7250 3750
-Wire Wire Line
-	7800 3300 7900 3300
-Wire Wire Line
-	7900 3300 7900 3400
-Wire Wire Line
-	7900 3400 8000 3400
-Wire Wire Line
-	8000 3600 7650 3600
-Wire Wire Line
-	7650 3600 7650 4450
-Wire Wire Line
-	7650 4450 6650 4450
-Text HLabel 5600 2200 1    50   Input ~ 0
-USB_DP
-Text HLabel 5500 2200 1    50   Input ~ 0
-USB_DM
 $Comp
 L Device:C C11
@@
 F 0 "C11" H 7165 2096 50  0000 L CNN
 F 1 "100μF" H 7165 2005 50  0000 L CNN
-F 2 "Capacitor_SMD:CP_Elec_4x3" H 7088 1900 50  0001 C CNN
-F 3 "~" H 7050 2050 50  0001 C CNN
+F 2 "Capacitor_SMD:C_1210_3225Metric" H 7088 1900 50  0001 C CNN
+F 3 "https://www.mouser.com/datasheet/2/40/TPS-2066671.pdf" H 7050 2050 50  0001 C CNN
+F 4 "AVX" H 7165 2196 50  0001 C CNN "Manufacturer_Name"
+F 5 "TPST107M004R0500" H 7165 2196 50  0001 C CNN "Manufacturer_Part_Number"
+F 6 "0.93" H 7165 2196 50  0001 C CNN "Price"
+F 7 "581-TPST107M004R0500" H 7165 2196 50  0001 C CNN "Vendor Part Number"
+F 8 "Mouser" H 7165 2196 50  0001 C CNN "Vendor"
 	1    7050 2050
 	1    0    0    -1
 $EndComp
-Wire Wire Line
-	7050 1900 6900 1900
-Connection ~ 6900 1900
-Wire Wire Line
-	6900 1900 6900 1800
 $Comp
 L power:GNDREF #PWR0129
@@
 	1    0    0    -1
 $EndComp
+Text Notes 5400 1700 0    50   ~ 0
+See HS-100B datasheet
+Text Notes 8100 3150 0    50   ~ 0
+See TX-500 adapters\nAudio data cable
+Text HLabel 5600 2200 1    50   Input ~ 0
+USB_DP
+Text HLabel 5500 2200 1    50   Input ~ 0
+USB_DM
+Wire Wire Line
+	6500 3350 6650 3350
+Wire Wire Line
+	6650 3350 6650 3650
+Wire Wire Line
+	6500 3650 6650 3650
+Wire Wire Line
+	6650 3650 6650 4450
+Wire Wire Line
+	6500 4450 6650 4450
+Wire Wire Line
+	6650 4450 6650 4650
+Wire Wire Line
+	4800 4450 4600 4450
+Wire Wire Line
+	6500 4150 7450 4150
+Wire Wire Line
+	7450 4150 7450 3500
+Wire Wire Line
+	7450 3500 8000 3500
+Wire Wire Line
+	6500 3950 7250 3950
+Wire Wire Line
+	7250 3950 7250 3750
+Wire Wire Line
+	6500 3750 7250 3750
+Wire Wire Line
+	6500 3450 6900 3450
+Wire Wire Line
+	6500 3550 6900 3550
+Wire Wire Line
+	6900 3550 6900 3450
+Wire Wire Line
+	6500 4050 6900 4050
+Wire Wire Line
+	6900 4050 6900 3550
+Wire Wire Line
+	5800 5250 5800 5400
+Wire Wire Line
+	5800 5400 4600 5400
+Wire Wire Line
+	4600 4450 4600 5400
+Wire Wire Line
+	4600 5400 4600 5500
+Wire Wire Line
+	4800 4250 4600 4250
+Wire Wire Line
+	4600 4250 4600 4450
+Wire Wire Line
+	4800 4050 4400 4050
+Wire Wire Line
+	4400 4050 4400 3850
+Wire Wire Line
+	4400 3850 4800 3850
+Wire Wire Line
+	5900 2550 5900 2350
+Wire Wire Line
+	5900 2350 6650 2350
+Wire Wire Line
+	6650 2350 6650 3350
+Wire Wire Line
+	7250 3300 7500 3300
+Wire Wire Line
+	7250 3300 7250 3750
+Wire Wire Line
+	7800 3300 7900 3300
+Wire Wire Line
+	7900 3300 7900 3400
+Wire Wire Line
+	7900 3400 8000 3400
+Wire Wire Line
+	8000 3600 7650 3600
+Wire Wire Line
+	7650 3600 7650 4450
+Wire Wire Line
+	7650 4450 6650 4450
+Wire Wire Line
+	7050 1900 6900 1900
+Wire Wire Line
+	6900 1900 6900 1800
 Wire Wire Line
 	6900 1900 6900 3450
+Wire Wire Line
+	5600 2200 5600 2550
+Wire Wire Line
+	5500 2200 5500 2550
+Connection ~ 6650 3650
+Connection ~ 6650 4450
+Connection ~ 7250 3750
+Connection ~ 6900 3550
+Connection ~ 4600 5400
+Connection ~ 4600 4450
+Connection ~ 6650 3350
+Connection ~ 6900 1900
 Connection ~ 6900 3450
-Wire Wire Line
-	5600 2200 5600 2550
-Wire Wire Line
-	5500 2200 5500 2550
 $EndSCHEMATC
