File: tx500-data.sch (KiCad schematic (older format))
At the start: 51 parts, among them J1 USB_B_Micro, J2 CAT, J3 REM/DATA, J4 USB_A, U1 TUSB2036, U2 FT232RL, U3 HS-100B, U4 TPS76333, U5 TPS2044D, U6 SN75240, U7 SN75240, Y1 6MHz

Commit message: Fix crystal BOM and footprint
Parts:
- Y1: footprint Crystal:Crystal_SMD_Abracon_ABM7-2Pin_6.0x3.5mm -> XT49M:XT49M; Manufacturer_Name ABRACON -> Vishay; Manufacturer_Part_Number AWSCR-6.00CPLA-C30-T4 -> XT9M20ANA6M; Price 0.36 -> 0.95; Vendor Part Number 815-CR-6.00CPLA-30-T -> 73-XT49M600-20
Changed lines of the file:
@@
 Sheet 1 1
 Title "TX-500 Data Interface"
-Date "2021-03-22"
-Rev "0.4"
+Date "2021-04-02"
+Rev "0.5"
 Comp "Chris Keller K0SWE"
 Comment1 "Licensed under Apache-2.0"
@@
 F 0 "Y1" H 1300 5018 50  0000 C CNN
 F 1 "6MHz" H 1300 4927 50  0000 C CNN
-F 2 "Crystal:Crystal_SMD_Abracon_ABM7-2Pin_6.0x3.5mm" H 1300 4750 50  0001 C CNN
+F 2 "XT49M:XT49M" H 1300 4750 50  0001 C CNN
 F 3 "https://www.mouser.com/datasheet/2/3/AWSCR-CPLA-1595603.pdf" H 1300 4750 50  0001 C CNN
 F 4 "Hub controller clock" H 1300 5118 50  0001 C CNN "Description"
-F 5 "ABRACON" H 1300 5118 50  0001 C CNN "Manufacturer_Name"
-F 6 "AWSCR-6.00CPLA-C30-T4" H 1300 5118 50  0001 C CNN "Manufacturer_Part_Number"
-F 7 "0.36" H 1300 5118 50  0001 C CNN "Price"
-F 8 "815-CR-6.00CPLA-30-T" H 1300 5118 50  0001 C CNN "Vendor Part Number"
+F 5 "Vishay" H 1300 5118 50  0001 C CNN "Manufacturer_Name"
+F 6 "XT9M20ANA6M" H 1300 5118 50  0001 C CNN "Manufacturer_Part_Number"
+F 7 "0.95" H 1300 5118 50  0001 C CNN "Price"
+F 8 "73-XT49M600-20" H 1300 5118 50  0001 C CNN "Vendor Part Number"
 F 9 "Mouser" H 1300 5118 50  0001 C CNN "Vendor"
 	1    1300 4750
@@
 P 1000 1500
 AR Path="/6057976E/6067467C" Ref="#PWR?"  Part="1"
-AR Path="/6067467C" Ref="#PWR?"  Part="1"
-F 0 "#PWR?" H 1000 1250 50  0001 C CNN
+AR Path="/6067467C" Ref="#PWR0103"  Part="1"
+F 0 "#PWR0103" H 1000 1250 50  0001 C CNN
 F 1 "GNDREF" H 1005 1327 50  0001 C CNN
 F 2 "" H 1000 1500 50  0001 C CNN
@@
 P 1400 1500
 AR Path="/6057976E/6069D36F" Ref="#PWR?"  Part="1"
-AR Path="/6069D36F" Ref="#PWR?"  Part="1"
-F 0 "#PWR?" H 1400 1250 50  0001 C CNN
+AR Path="/6069D36F" Ref="#PWR0104"  Part="1"
+F 0 "#PWR0104" H 1400 1250 50  0001 C CNN
 F 1 "GNDREF" H 1405 1327 50  0001 C CNN
 F 2 "" H 1400 1500 50  0001 C CNN
@@
 P 2250 1500
 AR Path="/6057976E/6069D89E" Ref="#PWR?"  Part="1"
-AR Path="/6069D89E" Ref="#PWR?"  Part="1"
-F 0 "#PWR?" H 2250 1250 50  0001 C CNN
+AR Path="/6069D89E" Ref="#PWR0109"  Part="1"
+F 0 "#PWR0109" H 2250 1250 50  0001 C CNN
 F 1 "GNDREF" H 2255 1327 50  0001 C CNN
 F 2 "" H 2250 1500 50  0001 C CNN
@@
 AR Path="/6057976E/6070717E" Ref="#PWR?"  Part="1"
 AR Path="/605B3ED2/6070717E" Ref="#PWR?"  Part="1"
-AR Path="/6070717E" Ref="#PWR?"  Part="1"
-F 0 "#PWR?" H 3400 7350 50  0001 C CNN
+AR Path="/6070717E" Ref="#PWR0114"  Part="1"
+F 0 "#PWR0114" H 3400 7350 50  0001 C CNN
 F 1 "GNDREF" H 3405 7427 50  0001 C CNN
 F 2 "" H 3400 7600 50  0001 C CNN

Commit message: Use standard footprint for crystal
Parts:
- Y1: footprint XT49M:XT49M -> Crystal:Crystal_SMD_HC49-SD
Changed lines of the file:
@@
 F 0 "Y1" H 1300 5018 50  0000 C CNN
 F 1 "6MHz" H 1300 4927 50  0000 C CNN
-F 2 "XT49M:XT49M" H 1300 4750 50  0001 C CNN
+F 2 "Crystal:Crystal_SMD_HC49-SD" H 1300 4750 50  0001 C CNN
 F 3 "https://www.mouser.com/datasheet/2/3/AWSCR-CPLA-1595603.pdf" H 1300 4750 50  0001 C CNN
 F 4 "Hub controller clock" H 1300 5118 50  0001 C CNN "Description"

Commit message: Use smaller dimensions capacitor
Parts:
- C1, C10, C2, C9: Description (none) -> -; quantity (none) -> 4
- C11, C16, C17: footprint Capacitor_SMD:C_1210_3225Metric -> 6TPE120MAZB:CAPPM3528X200N; symbol Device:C -> Device:CP; Description (none) -> -; Manufacturer_Name (none) -> Panasonic; Manufacturer_Part_Number (none) -> 6TPE120MAZB; Price (none) -> 1.3; Vendor (none) -> Mouser; Vendor Part Number (none) -> 667-6TPE120MAZB; quantity (none) -> 3
- C12, R17: Description (none) -> -; quantity (none) -> 1
- C13, C14, C18, C3, R1, R4: Description (none) -> -; quantity (none) -> 2
- C15, C20, C4: Description (none) -> -; quantity (none) -> 3
- J1: Description (none) -> Upstream USB socket; Manufacturer_Name (none) -> Molex; Manufacturer_Part_Number (none) -> 47346-0001; Price (none) -> 0.95; Vendor (none) -> Mouser; Vendor Part Number (none) -> 538-47346-0001; quantity (none) -> 1
- J2, J3, J4, U1, U2, U3, U4, Y1: quantity (none) -> 1
- R10, R2, R3, R5, R6, R7, R8, R9: Description (none) -> -; quantity (none) -> 8
- R11, R12, R13, R14, R15, R16, R18: Description (none) -> -; quantity (none) -> 7
- R19, R20: Description (none) -> -; Manufacturer_Name (none) -> KOA Speer; Manufacturer_Part_Number (none) -> RK73Z2ETTD; Price (none) -> 0.14; Vendor (none) -> Mouser; Vendor Part Number (none) -> 660-RK73Z2ETTD; quantity (none) -> 2
- U5: Description (none) -> Overcurrent protection; Manufacturer_Name (none) -> TI; Manufacturer_Part_Number (none) -> TPS2044D; Price (none) -> 2.73; Vendor (none) -> Mouser; Vendor Part Number (none) -> 595-TPS2044BDR; quantity (none) -> 1
- U6, U7: Description (none) -> ESD protection; Manufacturer_Name (none) -> TI; Manufacturer_Part_Number (none) -> SN75240; Price (none) -> 1.31; Vendor (none) -> Mouser; Vendor Part Number (none) -> 595-SN75240PWR; quantity (none) -> 2
