File: tx500-data.sch (KiCad schematic (older format))
At the start: 69 parts, among them J1 USB_C_Receptacle, J2 FTDI, J3 AUDIO, SW1 VCCIO, U1 TUSB2036, U2 FT232RL, U3 HS-100B, U4 TPS76333, U5 SN75240, U6 TPS2041, Y1 AWSCR-6.00CPLA

Commit message: Add bulkhead parts to schematic
Parts:
- J2: value FTDI -> CAT; symbol Connector_Generic:Conn_01x06 -> Connector:Conn_01x06_Male
- J3: symbol Connector_Generic:Conn_01x06 -> Connector:Conn_01x06_Male
Connections:
- no-connect marks 29 -> 38
Other:
- note added: "Bulkhead Pigtail for AUDIO"
- note added: "Bulkhead Pigtail for CAT"
- moved on the sheet: C10, C11, C12, C13, C14, C15, C16, C17, C18, C7, C8, C9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
